File: hardware/kicad/Dual_Band_RFID_Reader/high_freq_rf.kicad_sch (KiCad schematic)
At the start: 23 parts, among them U4 MFRC522, Y1 Crystal

Commit message: move sheet template to kicad project folder
Parts:
- C10, C11, C12, C13, C14, C15, C16, C17, C18, C19, C20, C7, C8, C9: footprint (none) -> Capacitor_SMD:C_0603_1608Metric_Pad1.08x0.95mm_HandSolder
- R11, R12, R13, R15: footprint (none) -> Resistor_SMD:R_0603_1608Metric_Pad0.98x0.95mm_HandSolder

Commit message: Remove IRQ hw line from MFRC522, it's not useful
Connections:
- removed net IRQ: U4.23 (IRQ)
Changed lines of the file:
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@@
-    (stroke (width 0) (type default))
-  )
-  (wire (pts (xy 46.99 101.6) (xy 60.96 101.6))
     (stroke (width 0) (type default))
   )
@@
   )
   (hierarchical_label "MISO" (shape input) (at 46.99 82.55 180) (fields_autoplaced)
-    (effects (font (size 1.27 1.27)) (justify right))
-  )
-  (hierarchical_label "IRQ" (shape input) (at 46.99 101.6 180) (fields_autoplaced)
     (effects (font (size 1.27 1.27)) (justify right))
   )
@@
       (effects (font (size 1.27 1.27)) hide)
     )
-    (pin "23")
     (pin "1")
     (pin "10")

Commit message: adding Mousa's board work to branch
Parts:
- L2, L3, L4: footprint (none) -> Inductor_SMD:L_0603_1608Metric_Pad1.05x0.95mm_HandSolder
- U4: footprint (none) -> MIFARE:QFN50P500X500X100-33N
- Y1: footprint (none) -> Capstone Footprint Lib:Crystal_SMD_3225-4Pin_3.2x2.5mm_HandSoldering; Digi-Key URL (none) -> https://www.digikey.com/en/products/detail/iqd-frequency-pr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; Digi-Key part number (none) -> 1923-LFXTAL062461R; datasheet URL (none) -> https://www.iqdfrequencyproducts.com/products/pn/LFXTAL0624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
Changed lines of the file:
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@@
   )
   (symbol (lib_id "pspice:INDUCTOR") (at 245.11 93.98 270) (unit 1)
-    (in_bom yes) (on_board yes) (fields_autoplaced)
+    (in_bom yes) (on_board no) (fields_autoplaced)
     (property "Reference" "L4" (id 0) (at 247.65 92.7099 90)
       (effects (font (size 1.27 1.27)) (justify left))
@@
       (effects (font (size 1.27 1.27)) (justify left))
     )
-    (property "Footprint" "" (id 2) (at 245.11 93.98 0)
+    (property "Footprint" "Inductor_SMD:L_0603_1608Metric_Pad1.05x0.95mm_HandSolder" (id 2) (at 245.11 93.98 0)
       (effects (font (size 1.27 1.27)) hide)
     )
@@
       (effects (font (size 1.27 1.27)))
     )
-    (property "Footprint" "" (id 2) (at 152.4 81.28 0)
+    (property "Footprint" "Inductor_SMD:L_0603_1608Metric_Pad1.05x0.95mm_HandSolder" (id 2) (at 152.4 81.28 0)
       (effects (font (size 1.27 1.27)) hide)
     )
@@
       (effects (font (size 1.27 1.27)))
     )
-    (property "Footprint" "" (id 2) (at 123.19 118.11 0)
-      (effects (font (size 1.27 1.27)) hide)
-    )
-    (property "Datasheet" "~" (id 3) (at 123.19 118.11 0)
+    (property "Footprint" "Capstone Footprint Lib:Crystal_SMD_3225-4Pin_3.2x2.5mm_HandSoldering" (id 2) (at 123.19 118.11 0)
+      (effects (font (size 1.27 1.27)) hide)
+    )
+    (property "Datasheet" "" (id 3) (at 123.19 118.11 0)
+      (effects (font (size 1.27 1.27)) hide)
+    )
+    (property "Digi-Key part number" "1923-LFXTAL062461R" (id 4) (at 123.19 118.11 0)
+      (effects (font (size 1.27 1.27)) hide)
+    )
+    (property "Digi-Key URL" "https://www.digikey.com/en/products/detail/iqd-frequency-products/LFXTAL062461Reel/10240450" (id 5) (at 123.19 118.11 0)
+      (effects (font (size 1.27 1.27)) hide)
+    )
+    (property "datasheet URL" "https://www.iqdfrequencyproducts.com/products/pn/LFXTAL062461REEL.pdf" (id 6) (at 123.19 118.11 0)
       (effects (font (size 1.27 1.27)) hide)
     )
@@
       (effects (font (size 1.27 1.27)))
     )
-    (property "Footprint" "" (id 2) (at 85.09 91.44 0)
+    (property "Footprint" "MIFARE:QFN50P500X500X100-33N" (id 2) (at 85.09 91.44 0)
       (effects (font (size 1.27 1.27)) hide)
     )
@@
       (effects (font (size 1.27 1.27)))
     )
-    (property "Footprint" "" (id 2) (at 152.4 106.68 0)
-      (effects (font (size 1.27 1.27)) hide)
-    )
+    (property "Footprint" "Inductor_SMD:L_0603_1608Metric_Pad1.05x0.95mm_HandSolder" (id 2) (at 152.4 106.68 0)
+      (effects (font (size 1.27 1.27)) hide)
+    )

Commit message: Board Layout WIP
* Added correct footprint for the components that were
  producing errors
* added HF antenna trace on board periphery
* added pads for the LF antenna coil to be connected later
* corrected all the DRC errors
* completed HF layout
Parts:
- removed L4: INDUCTOR, Inductor_SMD:L_0603_1608Metric_Pad1.05x0.95mm_HandSolder, symbol pspice:INDUCTOR
- L2, L3: footprint Inductor_SMD:L_0603_1608Metric_Pad1.05x0.95mm_HandSolder -> Inductor_SMD:L_1210_3225Metric_Pad1.42x2.65mm_HandSolder
- U4: footprint MIFARE:QFN50P500X500X100-33N -> Package_DFN_QFN:QFN-32-1EP_5x5mm_P0.5mm_EP3.3x3.3mm; symbol capstone:MFRC522 -> Capstone Symbol Lib:MFRC522
Connections:
- net at C10.1, C15.1, C16.2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: now also R12.1, R13.1
- net at L2.1: now also U4.13 (TX2); no longer U4.11 (TX1)
- net at C7.1, U4.21 (OSCIN): now also Y1.3; no longer Y1.2
- net at L3.1: now also U4.11 (TX1); no longer U4.13 (TX2)
Changed lines of the file:
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@@
   (junction (at 222.25 93.98) (diameter 0) (color 0 0 0 0)
   )
+  (junction (at 245.11 93.98) (diameter 0) (color 0 0 0 0)
+  )
   (junction (at 85.09 58.42) (diameter 0) (color 0 0 0 0)
   )
@@
     (stroke (width 0) (type default))
   )
-  (wire (pts (xy 245.11 87.63) (xy 245.11 81.28))
-    (stroke (width 0) (type default))
-  )
   (wire (pts (xy 166.37 88.9) (xy 166.37 93.98))
     (stroke (width 0) (type default))
@@
     (stroke (width 0) (type default))
   )
+  (polyline (pts (xy 240.03 86.36) (xy 255.27 86.36))
+    (stroke (width 0) (type default))
+  )
   (wire (pts (xy 123.19 134.62) (xy 123.19 137.16))
     (stroke (width 0) (type default))
@@
     (stroke (width 0) (type default))
   )
+  (polyline (pts (xy 240.03 102.87) (xy 255.27 102.87))
+    (stroke (width 0) (type default))
+  )
   (wire (pts (xy 46.99 90.17) (xy 60.96 90.17))
     (stroke (width 0) (type default))
@@
     (stroke (width 0) (type default))
   )
-  (polyline (pts (xy 238.76 86.36) (xy 238.76 102.87))
-    (stroke (width 0) (type default))
-  )
-  (polyline (pts (xy 238.76 86.36) (xy 260.35 86.36))
-    (stroke (width 0) (type default))
-  )
-  (polyline (pts (xy 260.35 86.36) (xy 260.35 102.87))
-    (stroke (width 0) (type default))
-  )
-  (polyline (pts (xy 260.35 102.87) (xy 238.76 102.87))
+  (polyline (pts (xy 240.03 86.36) (xy 240.03 102.87))
+    (stroke (width 0) (type default))
+  )
+  (polyline (pts (xy 255.27 86.36) (xy 255.27 102.87))
     (stroke (width 0) (type default))
   )
@@
     (stroke (width 0) (type default))
   )
+  (wire (pts (xy 245.11 93.98) (xy 245.11 106.68))
+    (stroke (width 0) (type default))
+  )
+  (wire (pts (xy 222.25 93.98) (xy 245.11 93.98))
+    (stroke (width 0) (type default))
+  )
   (wire (pts (xy 106.68 86.36) (xy 114.3 86.36))
     (stroke (width 0) (type default))
@@
     (stroke (width 0) (type default))
   )
+  (polyline (pts (xy 254 86.36) (xy 254 86.36))
+    (stroke (width 0) (type default))
+  )
   (wire (pts (xy 241.3 106.68) (xy 245.11 106.68))
     (stroke (width 0) (type default))
   )
-  (wire (pts (xy 245.11 100.33) (xy 245.11 106.68))
-    (stroke (width 0) (type default))
-  )
   (wire (pts (xy 166.37 81.28) (xy 200.66 81.28))
     (stroke (width 0) (type default))
@@
   )
   (wire (pts (xy 92.71 120.65) (xy 88.9 120.65))
+    (stroke (width 0) (type default))
+  )
+  (wire (pts (xy 245.11 81.28) (xy 245.11 93.98))
     (stroke (width 0) (type default))
   )
@@
     (effects (font (size 2.54 2.54)) (justify left bottom))
   )
-  (text "PCB Antenna\nTrace" (at 248.92 111.76 0)
-    (effects (font (size 2.54 2.54)) (justify left bottom))
+  (text "PCB Antenna\nTrace" (at 247.65 109.22 0)
+    (effects (font (size 1.778 1.778)) (justify left bottom))
   )
   (hierarchical_label "SCK" (shape input) (at 46.99 90.17 180) (fields_autoplaced)
@@
     (pin "2")
   )
-  (symbol (lib_id "pspice:INDUCTOR") (at 245.11 93.98 270) (unit 1)
-    (in_bom yes) (on_board no) (fields_autoplaced)
-    (property "Reference" "L4" (id 0) (at 247.65 92.7099 90)
-      (effects (font (size 1.27 1.27)) (justify left))
-    )
-    (property "Value" "INDUCTOR" (id 1) (at 247.65 95.2499 90)
-      (effects (font (size 1.27 1.27)) (justify left))
-    )
-    (property "Footprint" "Inductor_SMD:L_0603_1608Metric_Pad1.05x0.95mm_HandSolder" (id 2) (at 245.11 93.98 0)
-      (effects (font (size 1.27 1.27)) hide)
-    )
-    (property "Datasheet" "~" (id 3) (at 245.11 93.98 0)
-      (effects (font (size 1.27 1.27)) hide)
-    )
-    (pin "1")
-    (pin "2")
-  )
   (symbol (lib_id "power:GND") (at 123.19 137.16 0) (unit 1)
     (in_bom yes) (on_board yes) (fields_autoplaced)
@@
       (effects (font (size 1.27 1.27)))
     )
-    (property "Footprint" "Inductor_SMD:L_0603_1608Metric_Pad1.05x0.95mm_HandSolder" (id 2) (at 152.4 81.28 0)
+    (property "Footprint" "Inductor_SMD:L_1210_3225Metric_Pad1.42x2.65mm_HandSolder" (id 2) (at 152.4 81.28 0)
       (effects (font (size 1.27 1.27)) hide)
     )
@@
       (effects (font (size 1.27 1.27)) hide)
     )
-    (property "Datasheet" "" (id 3) (at 123.19 118.11 0)
+    (property "Datasheet" "~" (id 3) (at 123.19 118.11 0)
       (effects (font (size 1.27 1.27)) hide)
     )
@@
     )
     (pin "1")
-    (pin "2")
+    (pin "3")
   )
   (symbol (lib_id "Device:C") (at 130.81 57.15 270) (unit 1)
@@
     (pin "2")
   )
-  (symbol (lib_id "capstone:MFRC522") (at 85.09 91.44 0) (unit 1)
+  (symbol (lib_id "Capstone Symbol Lib:MFRC522") (at 85.09 91.44 0) (unit 1)
     (in_bom yes) (on_board yes) (fields_autoplaced)
     (property "Reference" "U4" (id 0) (at 83.82 67.31 0)
@@
       (effects (font (size 1.27 1.27)))
     )
-    (property "Footprint" "MIFARE:QFN50P500X500X100-33N" (id 2) (at 85.09 91.44 0)
+    (property "Footprint" "Package_DFN_QFN:QFN-32-1EP_5x5mm_P0.5mm_EP3.3x3.3mm" (id 2) (at 85.09 91.44 0)
       (effects (font (size 1.27 1.27)) hide)
     )
@@
       (effects (font (size 1.27 1.27)))
     )
-    (property "Footprint" "Inductor_SMD:L_0603_1608Metric_Pad1.05x0.95mm_HandSolder" (id 2) (at 152.4 106.68 0)
-      (effects (font (size 1.27 1.27)) hide)
-    )
+    (property "Footprint" "Inductor_SMD:L_1210_3225Metric_Pad1.42x2.65mm_HandSolder" (id 2) (at 152.4 106.68 0)
+      (effects (font (size 1.27 1.27)) hide)
+    )

Commit message: Updates traces
Parts:
- added L4: INDUCTOR, Inductor_SMD:L_0603_1608Metric_Pad1.05x0.95mm_HandSolder, symbol pspice:INDUCTOR
- L2, L3: footprint Inductor_SMD:L_1210_3225Metric_Pad1.42x2.65mm_HandSolder -> Inductor_SMD:L_0603_1608Metric_Pad1.05x0.95mm_HandSolder
- U4: footprint Package_DFN_QFN:QFN-32-1EP_5x5mm_P0.5mm_EP3.3x3.3mm -> MIFARE:QFN50P500X500X100-33N; symbol Capstone Symbol Lib:MFRC522 -> capstone:MFRC522
- Y1: footprint Capstone Footprint Lib:Crystal_SMD_3225-4Pin_3.2x2.5mm_HandSoldering -> Crystal:Crystal_SMD_HC49-SD_HandSoldering; Digi-Key URL https://www.digikey.com/en/products/detail/iqd-frequency-pr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 -> (none); Digi-Key part number 1923-LFXTAL062461R -> (none); datasheet URL https://www.iqdfrequencyproducts.com/products/pn/LFXTAL0624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 -> (none)
Connections:
- net at C10.1, C15.1, C16.2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: no longer R12.1, R13.1
- net at L2.1: now also U4.11 (TX1); no longer U4.13 (TX2)
- net at C7.1, U4.21 (OSCIN): now also Y1.2; no longer Y1.3
- net at L3.1: now also U4.13 (TX2); no longer U4.11 (TX1)
- new net: L4.1, R12.1
- new net: L4.2, R13.1
Changed lines of the file:
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@@
   (junction (at 222.25 93.98) (diameter 0) (color 0 0 0 0)
   )
-  (junction (at 245.11 93.98) (diameter 0) (color 0 0 0 0)
-  )
   (junction (at 85.09 58.42) (diameter 0) (color 0 0 0 0)
   )
@@
     (stroke (width 0) (type default))
   )
+  (wire (pts (xy 245.11 87.63) (xy 245.11 81.28))
+    (stroke (width 0) (type default))
+  )
   (wire (pts (xy 166.37 88.9) (xy 166.37 93.98))
     (stroke (width 0) (type default))
@@
     (stroke (width 0) (type default))
   )
-  (polyline (pts (xy 240.03 86.36) (xy 255.27 86.36))
-    (stroke (width 0) (type default))
-  )
   (wire (pts (xy 123.19 134.62) (xy 123.19 137.16))
     (stroke (width 0) (type default))
@@
     (stroke (width 0) (type default))
   )
-  (polyline (pts (xy 240.03 102.87) (xy 255.27 102.87))
-    (stroke (width 0) (type default))
-  )
   (wire (pts (xy 46.99 90.17) (xy 60.96 90.17))
     (stroke (width 0) (type default))
@@
     (stroke (width 0) (type default))
   )
-  (polyline (pts (xy 240.03 86.36) (xy 240.03 102.87))
-    (stroke (width 0) (type default))
-  )
-  (polyline (pts (xy 255.27 86.36) (xy 255.27 102.87))
+  (polyline (pts (xy 238.76 86.36) (xy 238.76 102.87))
+    (stroke (width 0) (type default))
+  )
+  (polyline (pts (xy 238.76 86.36) (xy 260.35 86.36))
+    (stroke (width 0) (type default))
+  )
+  (polyline (pts (xy 260.35 86.36) (xy 260.35 102.87))
+    (stroke (width 0) (type default))
+  )
+  (polyline (pts (xy 260.35 102.87) (xy 238.76 102.87))
     (stroke (width 0) (type default))
   )
@@
     (stroke (width 0) (type default))
   )
-  (wire (pts (xy 245.11 93.98) (xy 245.11 106.68))
-    (stroke (width 0) (type default))
-  )
-  (wire (pts (xy 222.25 93.98) (xy 245.11 93.98))
-    (stroke (width 0) (type default))
-  )
   (wire (pts (xy 106.68 86.36) (xy 114.3 86.36))
     (stroke (width 0) (type default))
@@
     (stroke (width 0) (type default))
   )
-  (polyline (pts (xy 254 86.36) (xy 254 86.36))
-    (stroke (width 0) (type default))
-  )
   (wire (pts (xy 241.3 106.68) (xy 245.11 106.68))
     (stroke (width 0) (type default))
   )
+  (wire (pts (xy 245.11 100.33) (xy 245.11 106.68))
+    (stroke (width 0) (type default))
+  )
   (wire (pts (xy 166.37 81.28) (xy 200.66 81.28))
     (stroke (width 0) (type default))
@@
   )
   (wire (pts (xy 92.71 120.65) (xy 88.9 120.65))
-    (stroke (width 0) (type default))
-  )
-  (wire (pts (xy 245.11 81.28) (xy 245.11 93.98))
     (stroke (width 0) (type default))
   )
@@
     (effects (font (size 2.54 2.54)) (justify left bottom))
   )
-  (text "PCB Antenna\nTrace" (at 247.65 109.22 0)
-    (effects (font (size 1.778 1.778)) (justify left bottom))
+  (text "PCB Antenna\nTrace" (at 248.92 111.76 0)
+    (effects (font (size 2.54 2.54)) (justify left bottom))
   )
   (hierarchical_label "SCK" (shape input) (at 46.99 90.17 180) (fields_autoplaced)
@@
     (pin "2")
   )
+  (symbol (lib_id "pspice:INDUCTOR") (at 245.11 93.98 270) (unit 1)
+    (in_bom yes) (on_board yes) (fields_autoplaced)
+    (property "Reference" "L4" (id 0) (at 247.65 92.7099 90)
+      (effects (font (size 1.27 1.27)) (justify left))
+    )
+    (property "Value" "INDUCTOR" (id 1) (at 247.65 95.2499 90)
+      (effects (font (size 1.27 1.27)) (justify left))
+    )
+    (property "Footprint" "Inductor_SMD:L_0603_1608Metric_Pad1.05x0.95mm_HandSolder" (id 2) (at 245.11 93.98 0)
+      (effects (font (size 1.27 1.27)) hide)
+    )
+    (property "Datasheet" "~" (id 3) (at 245.11 93.98 0)
+      (effects (font (size 1.27 1.27)) hide)
+    )
+    (pin "1")
+    (pin "2")
+  )
   (symbol (lib_id "power:GND") (at 123.19 137.16 0) (unit 1)
     (in_bom yes) (on_board yes) (fields_autoplaced)
@@
       (effects (font (size 1.27 1.27)))
     )
-    (property "Footprint" "Inductor_SMD:L_1210_3225Metric_Pad1.42x2.65mm_HandSolder" (id 2) (at 152.4 81.28 0)
+    (property "Footprint" "Inductor_SMD:L_0603_1608Metric_Pad1.05x0.95mm_HandSolder" (id 2) (at 152.4 81.28 0)
       (effects (font (size 1.27 1.27)) hide)
     )
@@
       (effects (font (size 1.27 1.27)))
     )
-    (property "Footprint" "Capstone Footprint Lib:Crystal_SMD_3225-4Pin_3.2x2.5mm_HandSoldering" (id 2) (at 123.19 118.11 0)
+    (property "Footprint" "Crystal:Crystal_SMD_HC49-SD_HandSoldering" (id 2) (at 123.19 118.11 0)
       (effects (font (size 1.27 1.27)) hide)
     )
@@
       (effects (font (size 1.27 1.27)) hide)
     )
-    (property "Digi-Key part number" "1923-LFXTAL062461R" (id 4) (at 123.19 118.11 0)
-      (effects (font (size 1.27 1.27)) hide)
-    )
-    (property "Digi-Key URL" "https://www.digikey.com/en/products/detail/iqd-frequency-products/LFXTAL062461Reel/10240450" (id 5) (at 123.19 118.11 0)
-      (effects (font (size 1.27 1.27)) hide)
-    )
-    (property "datasheet URL" "https://www.iqdfrequencyproducts.com/products/pn/LFXTAL062461REEL.pdf" (id 6) (at 123.19 118.11 0)
-      (effects (font (size 1.27 1.27)) hide)
-    )
-    (pin "1")
-    (pin "3")
+    (pin "1")
+    (pin "2")
   )
   (symbol (lib_id "Device:C") (at 130.81 57.15 270) (unit 1)
@@
     (pin "2")
   )
-  (symbol (lib_id "Capstone Symbol Lib:MFRC522") (at 85.09 91.44 0) (unit 1)
+  (symbol (lib_id "capstone:MFRC522") (at 85.09 91.44 0) (unit 1)
     (in_bom yes) (on_board yes) (fields_autoplaced)
     (property "Reference" "U4" (id 0) (at 83.82 67.31 0)
@@
       (effects (font (size 1.27 1.27)))
     )
-    (property "Footprint" "Package_DFN_QFN:QFN-32-1EP_5x5mm_P0.5mm_EP3.3x3.3mm" (id 2) (at 85.09 91.44 0)
+    (property "Footprint" "MIFARE:QFN50P500X500X100-33N" (id 2) (at 85.09 91.44 0)
       (effects (font (size 1.27 1.27)) hide)
     )
@@
       (effects (font (size 1.27 1.27)))
     )
-    (property "Footprint" "Inductor_SMD:L_1210_3225Metric_Pad1.42x2.65mm_HandSolder" (id 2) (at 152.4 106.68 0)
-      (effects (font (size 1.27 1.27)) hide)
-    )
+    (property "Footprint" "Inductor_SMD:L_0603_1608Metric_Pad1.05x0.95mm_HandSolder" (id 2) (at 152.4 106.68 0)
+      (effects (font (size 1.27 1.27)) hide)
+    )
