File: hardware/kicad/Labpass RFID Reader/LF_RF.kicad_sch (KiCad schematic)
At the start: 23 parts, among them U2 LM393, U3 LM324

Commit message: Add terminal block for gpio to ext relay
Parts:
- J3: value (none) -> Conn_01x02; footprint (none) -> Connector_PinHeader_2.54mm:PinHeader_1x02_P2.54mm_Horizontal
- R2: value (none) -> 220k; footprint (none) -> Resistor_SMD:R_0603_1608Metric
- R3: value (none) -> 47k; footprint (none) -> Resistor_SMD:R_0603_1608Metric
- R7: value (none) -> 82k; footprint (none) -> Resistor_SMD:R_0603_1608Metric
- RV1, RV2: value (none) -> 50k; footprint (none) -> Capstone Footprint Library:TC33X
- U2: value (none) -> LM393; footprint (none) -> Package_SO:SOIC-8_3.9x4.9mm_P1.27mm
- U3: value (none) -> LM324; footprint (none) -> Package_SO:SO-14_3.9x8.65mm_P1.27mm
Changed lines of the file:
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@@
       (effects (font (size 1.27 1.27)) (justify left))
     )
-    (property "Value" "" (id 1) (at 147.32 104.1399 0)
-      (effects (font (size 1.27 1.27)) (justify left))
-    )
-    (property "Footprint" "" (id 2) (at 145.796 103.124 90)
+    (property "Value" "82k" (id 1) (at 147.32 104.1399 0)
+      (effects (font (size 1.27 1.27)) (justify left))
+    )
+    (property "Footprint" "Resistor_SMD:R_0603_1608Metric" (id 2) (at 145.796 103.124 90)
       (effects (font (size 1.27 1.27)) hide)
     )
@@
       (effects (font (size 1.27 1.27)) (justify left))
     )
-    (property "Value" "" (id 1) (at 123.19 67.3099 0)
-      (effects (font (size 1.27 1.27)) (justify left))
-    )
-    (property "Footprint" "" (id 2) (at 123.19 63.5 0)
+    (property "Value" "LM324" (id 1) (at 123.19 67.3099 0)
+      (effects (font (size 1.27 1.27)) (justify left))
+    )
+    (property "Footprint" "Package_SO:SO-14_3.9x8.65mm_P1.27mm" (id 2) (at 123.19 63.5 0)
       (effects (font (size 1.27 1.27)) hide)
     )
@@
       (effects (font (size 1.27 1.27)) (justify left))
     )
-    (property "Value" "" (id 1) (at 104.14 126.9999 0)
-      (effects (font (size 1.27 1.27)) (justify left))
-    )
-    (property "Footprint" "" (id 2) (at 102.616 125.984 90)
+    (property "Value" "47k" (id 1) (at 104.14 126.9999 0)
+      (effects (font (size 1.27 1.27)) (justify left))
+    )
+    (property "Footprint" "Resistor_SMD:R_0603_1608Metric" (id 2) (at 102.616 125.984 90)
       (effects (font (size 1.27 1.27)) hide)
     )
@@
     (in_bom yes) (on_board yes)
     (property "Reference" "U3" (id 0) (at 119.38 168.91 0))
-    (property "Value" "" (id 1) (at 119.38 171.45 0))
-    (property "Footprint" "" (id 2) (at 123.19 173.99 0)
+    (property "Value" "LM324" (id 1) (at 119.38 171.45 0))
+    (property "Footprint" "Package_SO:SO-14_3.9x8.65mm_P1.27mm" (id 2) (at 123.19 173.99 0)
       (effects (font (size 1.27 1.27)) hide)
     )
@@
       (effects (font (size 1.27 1.27)) (justify right) hide)
     )
-    (property "Value" "" (id 1) (at 99.06 140.9699 0)
-      (effects (font (size 1.27 1.27)) (justify right))
-    )
-    (property "Footprint" "" (id 2) (at 101.6 139.7 0)
+    (property "Value" "50k" (id 1) (at 99.06 140.9699 0)
+      (effects (font (size 1.27 1.27)) (justify right))
+    )
+    (property "Footprint" "Capstone Footprint Library:TC33X" (id 2) (at 101.6 139.7 0)
       (effects (font (size 1.27 1.27)) hide)
     )
@@
       (effects (font (size 1.27 1.27)) (justify left))
     )
-    (property "Value" "" (id 1) (at 90.17 67.3099 0)
-      (effects (font (size 1.27 1.27)) (justify left))
-    )
-    (property "Footprint" "" (id 2) (at 91.44 66.04 0)
+    (property "Value" "LM393" (id 1) (at 90.17 67.3099 0)
+      (effects (font (size 1.27 1.27)) (justify left))
+    )
+    (property "Footprint" "Package_SO:SOIC-8_3.9x4.9mm_P1.27mm" (id 2) (at 91.44 66.04 0)
       (effects (font (size 1.27 1.27)) hide)
     )
@@
     (in_bom yes) (on_board yes)
     (property "Reference" "U3" (id 0) (at 119.38 153.67 0))
-    (property "Value" "" (id 1) (at 119.38 156.21 0))
-    (property "Footprint" "" (id 2) (at 123.19 158.75 0)
+    (property "Value" "LM324" (id 1) (at 119.38 156.21 0))
+    (property "Footprint" "Package_SO:SO-14_3.9x8.65mm_P1.27mm" (id 2) (at 123.19 158.75 0)
       (effects (font (size 1.27 1.27)) hide)
     )
@@
     (in_bom yes) (on_board yes)
     (property "Reference" "U3" (id 0) (at 119.38 182.88 0))
-    (property "Value" "" (id 1) (at 119.38 185.42 0))
-    (property "Footprint" "" (id 2) (at 123.19 187.96 0)
+    (property "Value" "LM324" (id 1) (at 119.38 185.42 0))
+    (property "Footprint" "Package_SO:SO-14_3.9x8.65mm_P1.27mm" (id 2) (at 123.19 187.96 0)
       (effects (font (size 1.27 1.27)) hide)
     )
@@
       (effects (font (size 1.27 1.27)) (justify left))
     )
-    (property "Value" "" (id 1) (at 104.14 114.3 0)
-      (effects (font (size 1.27 1.27)) (justify left))
-    )
-    (property "Footprint" "" (id 2) (at 102.616 113.284 90)
+    (property "Value" "220k" (id 1) (at 104.14 114.3 0)
+      (effects (font (size 1.27 1.27)) (justify left))
+    )
+    (property "Footprint" "Resistor_SMD:R_0603_1608Metric" (id 2) (at 102.616 113.284 90)
       (effects (font (size 1.27 1.27)) hide)
     )
@@
     (in_bom yes) (on_board yes) (fields_autoplaced)
     (property "Reference" "U2" (id 0) (at 88.9 151.13 0))
-    (property "Value" "" (id 1) (at 88.9 153.67 0))
-    (property "Footprint" "" (id 2) (at 88.9 161.29 0)
+    (property "Value" "LM393" (id 1) (at 88.9 153.67 0))
+    (property "Footprint" "Package_SO:SOIC-8_3.9x4.9mm_P1.27mm" (id 2) (at 88.9 161.29 0)
       (effects (font (size 1.27 1.27)) hide)
     )
@@
       (effects (font (size 1.27 1.27)) (justify left))
     )
-    (property "Value" "" (id 1) (at 238.76 73.6599 0)
+    (property "Value" "Conn_01x02" (id 1) (at 238.76 73.6599 0)
       (effects (font (size 1.27 1.27)) (justify left) hide)
     )
-    (property "Footprint" "" (id 2) (at 236.22 71.12 0)
+    (property "Footprint" "Connector_PinHeader_2.54mm:PinHeader_1x02_P2.54mm_Horizontal" (id 2) (at 236.22 71.12 0)
       (effects (font (size 1.27 1.27)) hide)
     )
@@
       (effects (font (size 1.27 1.27)) (justify right))
     )
-    (property "Value" "" (id 1) (at 142.24 115.5699 0)
-      (effects (font (size 1.27 1.27)) (justify right))
-    )
-    (property "Footprint" "" (id 2) (at 144.78 115.57 0)
-      (effects (font (size 1.27 1.27)) hide)
-    )
+    (property "Value" "50k" (id 1) (at 142.24 115.5699 0)
+      (effects (font (size 1.27 1.27)) (justify right))
+    )
+    (property "Footprint" "Capstone Footprint Library:TC33X" (id 2) (at 144.78 115.57 0)
+      (effects (font (size 1.27 1.27)) hide)
+    )
