File: hardware/kicad/Labpass RFID Reader/Labpass RFID Reader.kicad_sch (KiCad schematic)
At the start: 1 part

Commit message: Add terminal block for gpio to ext relay
Connections:
- net Indicators/EXT_RELAY: now reaches U1.22
- net Indicators/buzzer renamed Indicators/BUZZER
- no-connect marks 10 -> 9
Other:
- sheet Indicators ports: added BUZZER, EXT_RELAY; removed buzzer
Changed lines of the file:
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@@
   (no_connect (at 119.38 129.54))
   (no_connect (at 119.38 127))
-  (no_connect (at 144.78 137.16))
   (no_connect (at 144.78 134.62))
   (no_connect (at 144.78 132.08))
@@
   )
   (wire (pts (xy 170.18 119.38) (xy 195.58 119.38))
+    (stroke (width 0) (type default) (color 0 0 0 0))
+  )
+  (wire (pts (xy 81.28 111.76) (xy 119.38 111.76))
     (stroke (width 0) (type default) (color 0 0 0 0))
   )
@@
       (effects (font (size 1.27 1.27)) (justify left top))
     )
-    (pin "buzzer" input (at 81.28 109.22 0)
+    (pin "BUZZER" input (at 81.28 109.22 0)
       (effects (font (size 1.27 1.27)) (justify right))
     )
@@
     )
     (pin "LED_2_B" input (at 81.28 93.98 0)
+      (effects (font (size 1.27 1.27)) (justify right))
+    )
+    (pin "EXT_RELAY" input (at 81.28 111.76 0)
       (effects (font (size 1.27 1.27)) (justify right))
     )
@@
       (reference "#PWR010") (unit 1) (value "GND") (footprint "")
     )
+    (path "/0302516d-709c-49c5-8a36-06b29a93bc66/0d2206eb-5bd8-442d-b04e-a22ed24a7013"
+      (reference "#PWR011") (unit 1) (value "GND") (footprint "")
+    )
     (path "/7edac1e6-8b57-42c3-be27-8045b1a8bdad/d661cc11-2696-47a1-a5ba-8072289e95c2"
       (reference "#PWR012") (unit 1) (value "GND") (footprint "")
@@
       (reference "J3") (unit 1) (value "Conn_01x02") (footprint "Connector_PinHeader_2.54mm:PinHeader_1x02_P2.54mm_Horizontal")
     )
+    (path "/0302516d-709c-49c5-8a36-06b29a93bc66/feb7af07-00c5-44ae-98db-c56bb3db2efb"
+      (reference "J4") (unit 1) (value "Conn_01x02") (footprint "Capstone Footprint Library:Anytek NQ")
+    )
     (path "/3c921900-5c38-4cb2-a335-20316312b0c1/e10d1f47-318e-4b6f-881f-5a81d1f14021"

Commit message: bump rev to 1.0.0
Parts:
- U1: value (none) -> adafruit_huzzah_32; footprint (none) -> Capstone Footprint Library:adafruit_huzzah_32
Changed lines of the file:
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@@
   (title_block
     (title "Labpass RFID Reader - MCU")
-    (date "2022-04-18")
-    (rev "0.1.0")
+    (date "2022-05-15")
+    (rev "1.0.0")
   )
   (junction (at 111.76 73.66) (diameter 0) (color 0 0 0 0)
@@
     (in_bom yes) (on_board yes)
     (property "Reference" "U1" (id 0) (at 132.08 114.3 0))
-    (property "Value" "" (id 1) (at 132.08 142.24 0))
-    (property "Footprint" "" (id 2) (at 129.54 113.03 0)
+    (property "Value" "adafruit_huzzah_32" (id 1) (at 132.08 142.24 0))
+    (property "Footprint" "Capstone Footprint Library:adafruit_huzzah_32" (id 2) (at 129.54 113.03 0)
       (effects (font (size 1.27 1.27)) hide)
     )
