File: hardware/kicad/Labpass RFID Reader - Mez/Labpass RFID Reader - Mez.kicad_pcb (KiCad board)
At the start: 2 copper layers, 61 x 70.1 mm, 15 parts, among them J1 Conn_01x03_Male

Commit message: Final rev 1.0.0
Parts:
- C1, C4: value 8-40p -> 11p
- C7, C8: value 8-40p -> 32p
Changed lines of the file:
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@@
       (effects (font (size 0.7 0.7) (thickness 0.1)))
     )
-    (fp_text value "8-40p" (at 0 1.43 180) (layer "F.Fab")
+    (fp_text value "11p" (at 0 1.43 180) (layer "F.Fab")
       (effects (font (size 1 1) (thickness 0.15)))
     )
@@
       (effects (font (size 0.7 0.7) (thickness 0.1)))
     )
-    (fp_text value "30p" (at -2.093 -0.046907 180) (layer "F.Fab")
+    (fp_text value "30p" (at -2.118 -0.821907 180) (layer "F.Fab")
       (effects (font (size 0.7 0.7) (thickness 0.1)))
     )
@@
       (effects (font (size 0.7 0.7) (thickness 0.1)))
     )
-    (fp_text value "8-40p" (at 2.182 -0.804 180) (layer "F.Fab")
-      (effects (font (size 0.7 0.7) (thickness 0.1)))
-    )
-    (fp_text user "${REFERENCE}" (at -0.043 -1.229 180) (layer "F.Fab")
+    (fp_text value "32p" (at 2.357 -0.779 180) (layer "F.Fab")
+      (effects (font (size 0.7 0.7) (thickness 0.1)))
+    )
+    (fp_text user "${REFERENCE}" (at -0.043 -1.229 180) (layer "F.Fab") hide
       (effects (font (size 0.7 0.7) (thickness 0.1)))
     )
@@
       (effects (font (size 0.7 0.7) (thickness 0.1)))
     )
-    (fp_text value "R_US" (at 0.028093 -1.057) (layer "F.Fab")
+    (fp_text value "R_US" (at -0.071907 -1.382) (layer "F.Fab")
       (effects (font (size 0.7 0.7) (thickness 0.1)))
     )
@@
       (effects (font (size 0.7 0.7) (thickness 0.1)))
     )
-    (fp_text value "8-40p" (at 0.225 -1.975) (layer "F.Fab")
-      (effects (font (size 0.7 0.7) (thickness 0.1)))
-    )
-    (fp_text user "${REFERENCE}" (at 0.025 -1.1) (layer "F.Fab")
+    (fp_text value "11p" (at 0.125 -1.525) (layer "F.Fab")
+      (effects (font (size 0.7 0.7) (thickness 0.1)))
+    )
+    (fp_text user "${REFERENCE}" (at 0.025 -1.1) (layer "F.Fab") hide
       (effects (font (size 0.7 0.7) (thickness 0.1)))
     )
@@
       (effects (font (size 0.7 0.7) (thickness 0.1)))
     )
-    (fp_text value "NC" (at -0.095 1.115) (layer "F.Fab")
+    (fp_text value "NC" (at -0.07 1.44) (layer "F.Fab")
       (effects (font (size 0.7 0.7) (thickness 0.1)))
     )
@@
       (effects (font (size 0.7 0.7) (thickness 0.1)))
     )
-    (fp_text value "R_US" (at -0.128093 1.107) (layer "F.Fab")
+    (fp_text value "R_US" (at -0.003093 1.507) (layer "F.Fab")
       (effects (font (size 0.7 0.7) (thickness 0.1)))
     )
@@
       (effects (font (size 0.7 0.7) (thickness 0.1)))
     )
-    (fp_text value "8-40p" (at -1.982 -1.095) (layer "F.Fab")
-      (effects (font (size 0.7 0.7) (thickness 0.1)))
-    )
-    (fp_text user "${REFERENCE}" (at 0.018 -1.17) (layer "F.Fab")
+    (fp_text value "32p" (at -2.507 -0.445) (layer "F.Fab")
+      (effects (font (size 0.7 0.7) (thickness 0.1)))
+    )
+    (fp_text user "${REFERENCE}" (at 0.018 -1.17) (layer "F.Fab") hide
       (effects (font (size 0.7 0.7) (thickness 0.1)))
     )
@@
       (effects (font (size 0.7 0.7) (thickness 0.1)))
     )
-    (fp_text value "30p" (at 1.893 -0.203093) (layer "F.Fab")
-      (effects (font (size 0.7 0.7) (thickness 0.1)))
-    )
+    (fp_text value "30p" (at 2.118 -0.403093) (layer "F.Fab")
+      (effects (font (size 0.7 0.7) (thickness 0.1)))
+    )
