File: hardware/kicad/Labpass RFID Reader - Mez/Labpass RFID Reader - Mez.kicad_sch (KiCad schematic)
At the start: 11 parts, among them J1 Conn_01x03_Male

Commit message: Polish reposition pin headers to clear mez board
Parts:
- C2, C3, C5, C6: footprint Capacitor_SMD:C_0201_0603Metric -> Capacitor_SMD:C_0603_1608Metric
- J1: symbol Connector:Conn_01x03_Male -> Connector_Generic:Conn_01x03
Other:
- note added: "Note: this 3-way short is really an inductive PCB trace but it must be done like this to be able to draw the board trace properly."
- title: (none) -> Labpass RFID Reader - Mezzanine
- moved on the sheet: C1, C2, C3, C4, C5, C6, C7, C8, R1, R2

Commit message: kicad backups
Parts:
- C1, C4, C7, C8: value C -> (none); footprint Capstone Footprint Library:JR400 -> (none)
- C2, C3: value C -> (none)
- C5, C6: value C -> (none); footprint Capacitor_SMD:C_0603_1608Metric -> (none)
- J1: value Conn_01x03_Male -> (none); footprint Connector_PinHeader_1.27mm:PinHeader_1x03_P1.27mm_Horizontal -> (none)
Changed lines of the file:
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@@
     (stroke (width 0) (type default) (color 0 0 0 0))
   )
-  (polyline (pts (xy 137.16 113.03) (xy 96.52 113.03))
+  (polyline (pts (xy 138.43 113.03) (xy 96.52 113.03))
     (stroke (width 0) (type default) (color 0 0 0 0))
   )
@@
     (stroke (width 0) (type default) (color 0 0 0 0))
   )
-  (polyline (pts (xy 137.16 62.23) (xy 137.16 113.03))
+  (polyline (pts (xy 138.43 62.23) (xy 138.43 113.03))
     (stroke (width 0) (type default) (color 0 0 0 0))
   )
@@
     (stroke (width 0) (type default) (color 0 0 0 0))
   )
-  (polyline (pts (xy 96.52 62.23) (xy 137.16 62.23))
+  (polyline (pts (xy 96.52 62.23) (xy 138.43 62.23))
     (stroke (width 0) (type default) (color 0 0 0 0))
   )
@@
     (in_bom yes) (on_board yes) (fields_autoplaced)
     (property "Reference" "C1" (id 0) (at 105.41 64.77 90))
-    (property "Value" "C" (id 1) (at 105.41 67.31 90))
-    (property "Footprint" "Capstone Footprint Library:JR400" (id 2) (at 105.41 72.39 0)
+    (property "Value" "" (id 1) (at 105.41 67.31 90))
+    (property "Footprint" "" (id 2) (at 105.41 72.39 0)
       (effects (font (size 1.27 1.27)) hide)
     )
@@
     (in_bom yes) (on_board yes)
     (property "Reference" "J1" (id 0) (at 86.36 81.28 0))
-    (property "Value" "Conn_01x03_Male" (id 1) (at 99.06 87.63 0)
-      (effects (font (size 1.27 1.27)) hide)
-    )
-    (property "Footprint" "Connector_PinHeader_1.27mm:PinHeader_1x03_P1.27mm_Horizontal" (id 2) (at 86.36 87.63 0)
+    (property "Value" "" (id 1) (at 99.06 87.63 0)
+      (effects (font (size 1.27 1.27)) hide)
+    )
+    (property "Footprint" "" (id 2) (at 86.36 87.63 0)
       (effects (font (size 1.27 1.27)) hide)
     )
@@
       (effects (font (size 1.27 1.27)) (justify right))
     )
-    (property "Value" "C" (id 1) (at 115.57 82.5499 0)
-      (effects (font (size 1.27 1.27)) (justify right))
-    )
-    (property "Footprint" "Capacitor_SMD:C_0603_1608Metric" (id 2) (at 120.3452 77.47 0)
+    (property "Value" "" (id 1) (at 115.57 82.5499 0)
+      (effects (font (size 1.27 1.27)) (justify right))
+    )
+    (property "Footprint" "" (id 2) (at 120.3452 77.47 0)
       (effects (font (size 1.27 1.27)) hide)
     )
@@
       (effects (font (size 1.27 1.27)) (justify left))
     )
-    (property "Value" "C" (id 1) (at 130.81 82.5499 0)
-      (effects (font (size 1.27 1.27)) (justify left))
-    )
-    (property "Footprint" "Capstone Footprint Library:JR400" (id 2) (at 127 81.28 0)
+    (property "Value" "" (id 1) (at 130.81 82.5499 0)
+      (effects (font (size 1.27 1.27)) (justify left))
+    )
+    (property "Footprint" "" (id 2) (at 127 81.28 0)
       (effects (font (size 1.27 1.27)) hide)
     )
@@
       (effects (font (size 1.27 1.27)) (justify left))
     )
-    (property "Value" "C" (id 1) (at 130.81 95.2499 0)
-      (effects (font (size 1.27 1.27)) (justify left))
-    )
-    (property "Footprint" "Capstone Footprint Library:JR400" (id 2) (at 127 93.98 0)
+    (property "Value" "" (id 1) (at 130.81 95.2499 0)
+      (effects (font (size 1.27 1.27)) (justify left))
+    )
+    (property "Footprint" "" (id 2) (at 127 93.98 0)
       (effects (font (size 1.27 1.27)) hide)
     )
@@
     (in_bom yes) (on_board yes)
     (property "Reference" "C4" (id 0) (at 105.41 107.95 90))
-    (property "Value" "C" (id 1) (at 105.41 110.49 90))
-    (property "Footprint" "Capstone Footprint Library:JR400" (id 2) (at 105.41 102.87 0)
+    (property "Value" "" (id 1) (at 105.41 110.49 90))
+    (property "Footprint" "" (id 2) (at 105.41 102.87 0)
       (effects (font (size 1.27 1.27)) hide)
     )
@@
       (effects (font (size 1.27 1.27)) (justify right))
     )
-    (property "Value" "C" (id 1) (at 115.57 95.2499 0)
-      (effects (font (size 1.27 1.27)) (justify right))
-    )
-    (property "Footprint" "Capacitor_SMD:C_0603_1608Metric" (id 2) (at 120.3452 90.17 0)
+    (property "Value" "" (id 1) (at 115.57 95.2499 0)
+      (effects (font (size 1.27 1.27)) (justify right))
+    )
+    (property "Footprint" "" (id 2) (at 120.3452 90.17 0)
       (effects (font (size 1.27 1.27)) hide)
     )
@@
     (in_bom yes) (on_board yes) (fields_autoplaced)
     (property "Reference" "C3" (id 0) (at 105.41 90.17 90))
-    (property "Value" "C" (id 1) (at 105.41 92.71 90))
+    (property "Value" "" (id 1) (at 105.41 92.71 90))
     (property "Footprint" "Capacitor_SMD:C_0603_1608Metric" (id 2) (at 109.22 96.8248 0)
       (effects (font (size 1.27 1.27)) hide)
@@
     (in_bom yes) (on_board yes)
     (property "Reference" "C2" (id 0) (at 105.41 82.55 90))
-    (property "Value" "C" (id 1) (at 105.41 85.09 90))
+    (property "Value" "" (id 1) (at 105.41 85.09 90))
     (property "Footprint" "Capacitor_SMD:C_0603_1608Metric" (id 2) (at 109.22 76.5048 0)
       (effects (font (size 1.27 1.27)) hide)
@@
   (symbol_instances
     (path "/02ab15cc-d4b2-48c5-a9cd-646284b23111"
-      (reference "C1") (unit 1) (value "C") (footprint "Capstone Footprint Library:JR400")
+      (reference "C1") (unit 1) (value "8-40p") (footprint "Capstone Footprint Library:JR400")
     )
     (path "/e2e20a04-e569-4b7b-a4f2-db2a07b068bb"
-      (reference "C2") (unit 1) (value "C") (footprint "Capacitor_SMD:C_0603_1608Metric")
+      (reference "C2") (unit 1) (value "NC") (footprint "Capacitor_SMD:C_0603_1608Metric")
     )
     (path "/e2ca6904-9e14-43f0-a6a5-38eb35c3f269"
-      (reference "C3") (unit 1) (value "C") (footprint "Capacitor_SMD:C_0603_1608Metric")
+      (reference "C3") (unit 1) (value "NC") (footprint "Capacitor_SMD:C_0603_1608Metric")
     )
     (path "/a97f35f9-349f-4c3a-b8b8-43d6d23efb6c"
-      (reference "C4") (unit 1) (value "C") (footprint "Capstone Footprint Library:JR400")
+      (reference "C4") (unit 1) (value "8-40p") (footprint "Capstone Footprint Library:JR400")
     )
     (path "/30827bd8-2c45-4b23-a780-e074789ebb44"
-      (reference "C5") (unit 1) (value "C") (footprint "Capacitor_SMD:C_0603_1608Metric")
+      (reference "C5") (unit 1) (value "30p") (footprint "Capacitor_SMD:C_0603_1608Metric")
     )
     (path "/d25c39f6-a172-4f2d-a9a2-d6403352ccfa"
-      (reference "C6") (unit 1) (value "C") (footprint "Capacitor_SMD:C_0603_1608Metric")
+      (reference "C6") (unit 1) (value "30p") (footprint "Capacitor_SMD:C_0603_1608Metric")
     )
     (path "/57084d4e-a4ea-4ca2-940d-82b7c846897f"
-      (reference "C7") (unit 1) (value "C") (footprint "Capstone Footprint Library:JR400")
+      (reference "C7") (unit 1) (value "8-40p") (footprint "Capstone Footprint Library:JR400")
     )
     (path "/8adc823a-7fcc-4921-9aae-eafe09355df0"
-      (reference "C8") (unit 1) (value "C") (footprint "Capstone Footprint Library:JR400")
+      (reference "C8") (unit 1) (value "8-40p") (footprint "Capstone Footprint Library:JR400")
     )
     (path "/2eda4bfe-b50d-4efe-b93a-e95f3e8ce559"
-      (reference "J1") (unit 1) (value "Conn_01x03_Male") (footprint "Connector_PinHeader_1.27mm:PinHeader_1x03_P1.27mm_Horizontal")
+      (reference "J1") (unit 1) (value "Conn_01x03_Male") (footprint "Capstone Footprint Library:PinHeader_1x03_P2.54mm_Horizontal")
     )
     (path "/d9a1c59d-f10b-4ac9-b0c2-f3f829909c8d"

Commit message: temp
Parts:
- C1, C4, C7, C8: symbol Device:C_Trim -> Device:C
- C2, C3: footprint Capacitor_SMD:C_0603_1608Metric -> (none)
- R1, R2: value R_US -> (none); footprint Resistor_SMD:R_0603_1608Metric -> (none)
Changed lines of the file:
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@@
     (effects (font (size 1.27 1.27)) (justify left bottom))
   )
-  (symbol (lib_id "Device:C_Trim") (at 105.41 72.39 90) (unit 1)
+  (symbol (lib_id "Device:C") (at 105.41 72.39 90) (unit 1)
     (in_bom yes) (on_board yes) (fields_autoplaced)
     (property "Reference" "C1" (id 0) (at 105.41 64.77 90))
     (property "Value" "" (id 1) (at 105.41 67.31 90))
-    (property "Footprint" "" (id 2) (at 105.41 72.39 0)
+    (property "Footprint" "" (id 2) (at 109.22 71.4248 0)
       (effects (font (size 1.27 1.27)) hide)
     )
@@
     (pin "2")
   )
-  (symbol (lib_id "Device:C_Trim") (at 127 81.28 0) (unit 1)
+  (symbol (lib_id "Device:C") (at 127 81.28 0) (unit 1)
     (in_bom yes) (on_board yes) (fields_autoplaced)
     (property "Reference" "C7" (id 0) (at 130.81 80.0099 0)
@@
       (effects (font (size 1.27 1.27)) (justify left))
     )
-    (property "Footprint" "" (id 2) (at 127 81.28 0)
+    (property "Footprint" "" (id 2) (at 127.9652 85.09 0)
       (effects (font (size 1.27 1.27)) hide)
     )
@@
     (pin "2")
   )
-  (symbol (lib_id "Device:C_Trim") (at 127 93.98 0) (unit 1)
+  (symbol (lib_id "Device:C") (at 127 93.98 0) (unit 1)
     (in_bom yes) (on_board yes) (fields_autoplaced)
     (property "Reference" "C8" (id 0) (at 130.81 92.7099 0)
@@
       (effects (font (size 1.27 1.27)) (justify left))
     )
-    (property "Footprint" "" (id 2) (at 127 93.98 0)
+    (property "Footprint" "" (id 2) (at 127.9652 97.79 0)
       (effects (font (size 1.27 1.27)) hide)
     )
@@
     (in_bom yes) (on_board yes) (fields_autoplaced)
     (property "Reference" "R2" (id 0) (at 143.51 91.44 90))
-    (property "Value" "R_US" (id 1) (at 143.51 93.98 90))
-    (property "Footprint" "Resistor_SMD:R_0603_1608Metric" (id 2) (at 143.764 96.774 90)
+    (property "Value" "" (id 1) (at 143.51 93.98 90))
+    (property "Footprint" "" (id 2) (at 143.764 96.774 90)
       (effects (font (size 1.27 1.27)) hide)
     )
@@
     (pin "2")
   )
-  (symbol (lib_id "Device:C_Trim") (at 105.41 102.87 90) (unit 1)
+  (symbol (lib_id "Device:C") (at 105.41 102.87 90) (unit 1)
     (in_bom yes) (on_board yes)
     (property "Reference" "C4" (id 0) (at 105.41 107.95 90))
     (property "Value" "" (id 1) (at 105.41 110.49 90))
-    (property "Footprint" "" (id 2) (at 105.41 102.87 0)
+    (property "Footprint" "" (id 2) (at 109.22 101.9048 0)
       (effects (font (size 1.27 1.27)) hide)
     )
@@
     (in_bom yes) (on_board yes) (fields_autoplaced)
     (property "Reference" "R1" (id 0) (at 143.51 71.12 90))
-    (property "Value" "R_US" (id 1) (at 143.51 73.66 90))
-    (property "Footprint" "Resistor_SMD:R_0603_1608Metric" (id 2) (at 143.764 76.454 90)
+    (property "Value" "" (id 1) (at 143.51 73.66 90))
+    (property "Footprint" "" (id 2) (at 143.764 76.454 90)
       (effects (font (size 1.27 1.27)) hide)
     )
@@
     (property "Reference" "C3" (id 0) (at 105.41 90.17 90))
     (property "Value" "" (id 1) (at 105.41 92.71 90))
-    (property "Footprint" "Capacitor_SMD:C_0603_1608Metric" (id 2) (at 109.22 96.8248 0)
+    (property "Footprint" "" (id 2) (at 109.22 96.8248 0)
       (effects (font (size 1.27 1.27)) hide)
     )
@@
     (property "Reference" "C2" (id 0) (at 105.41 82.55 90))
     (property "Value" "" (id 1) (at 105.41 85.09 90))
-    (property "Footprint" "Capacitor_SMD:C_0603_1608Metric" (id 2) (at 109.22 76.5048 0)
+    (property "Footprint" "" (id 2) (at 109.22 76.5048 0)
       (effects (font (size 1.27 1.27)) hide)
     )
@@
   (symbol_instances
     (path "/02ab15cc-d4b2-48c5-a9cd-646284b23111"
-      (reference "C1") (unit 1) (value "8-40p") (footprint "Capstone Footprint Library:JR400")
+      (reference "C1") (unit 1) (value "8-40p") (footprint "Resistor_SMD:R_0603_1608Metric")
     )
     (path "/e2e20a04-e569-4b7b-a4f2-db2a07b068bb"
@@
     )
     (path "/a97f35f9-349f-4c3a-b8b8-43d6d23efb6c"
-      (reference "C4") (unit 1) (value "8-40p") (footprint "Capstone Footprint Library:JR400")
+      (reference "C4") (unit 1) (value "8-40p") (footprint "Capacitor_SMD:C_0603_1608Metric")
     )
     (path "/30827bd8-2c45-4b23-a780-e074789ebb44"
@@
     )
     (path "/57084d4e-a4ea-4ca2-940d-82b7c846897f"
-      (reference "C7") (unit 1) (value "8-40p") (footprint "Capstone Footprint Library:JR400")
+      (reference "C7") (unit 1) (value "8-40p") (footprint "Capacitor_SMD:C_0603_1608Metric")
     )
     (path "/8adc823a-7fcc-4921-9aae-eafe09355df0"
-      (reference "C8") (unit 1) (value "8-40p") (footprint "Capstone Footprint Library:JR400")
+      (reference "C8") (unit 1) (value "8-40p") (footprint "Capacitor_SMD:C_0603_1608Metric")
     )
     (path "/2eda4bfe-b50d-4efe-b93a-e95f3e8ce559"

Commit message: bump rev to 1.0.0
Parts:
- C1: value (none) -> 8-40p; footprint (none) -> Resistor_SMD:R_0603_1608Metric
- C2, C3: value (none) -> NC; footprint (none) -> Capacitor_SMD:C_0603_1608Metric
- C4, C7, C8: value (none) -> 8-40p; footprint (none) -> Capacitor_SMD:C_0603_1608Metric
- C5, C6: value (none) -> 30p; footprint (none) -> Capacitor_SMD:C_0603_1608Metric
- J1: value (none) -> Conn_01x03_Male; footprint (none) -> Capstone Footprint Library:PinHeader_1x03_P2.54mm_Horizontal
- R1, R2: value (none) -> R_US; footprint (none) -> Resistor_SMD:R_0603_1608Metric
Changed lines of the file:
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@@
   (title_block
     (title "Labpass RFID Reader - Mezzanine")
-    (date "2022-04-18")
+    (date "2022-05-15")
+    (rev "1.0.0")
   )
   (junction (at 119.38 87.63) (diameter 0) (color 0 0 0 0)
@@
     (in_bom yes) (on_board yes) (fields_autoplaced)
     (property "Reference" "C1" (id 0) (at 105.41 64.77 90))
-    (property "Value" "" (id 1) (at 105.41 67.31 90))
-    (property "Footprint" "" (id 2) (at 109.22 71.4248 0)
+    (property "Value" "8-40p" (id 1) (at 105.41 67.31 90))
+    (property "Footprint" "Resistor_SMD:R_0603_1608Metric" (id 2) (at 109.22 71.4248 0)
       (effects (font (size 1.27 1.27)) hide)
     )
@@
     (in_bom yes) (on_board yes)
     (property "Reference" "J1" (id 0) (at 86.36 81.28 0))
-    (property "Value" "" (id 1) (at 99.06 87.63 0)
-      (effects (font (size 1.27 1.27)) hide)
-    )
-    (property "Footprint" "" (id 2) (at 86.36 87.63 0)
+    (property "Value" "Conn_01x03_Male" (id 1) (at 99.06 87.63 0)
+      (effects (font (size 1.27 1.27)) hide)
+    )
+    (property "Footprint" "Capstone Footprint Library:PinHeader_1x03_P2.54mm_Horizontal" (id 2) (at 86.36 87.63 0)
       (effects (font (size 1.27 1.27)) hide)
     )
@@
       (effects (font (size 1.27 1.27)) (justify right))
     )
-    (property "Value" "" (id 1) (at 115.57 82.5499 0)
+    (property "Value" "30p" (id 1) (at 115.57 82.5499 0)
       (effects (font (size 1.27 1.27)) (justify right))
     )
-    (property "Footprint" "" (id 2) (at 120.3452 77.47 0)
+    (property "Footprint" "Capacitor_SMD:C_0603_1608Metric" (id 2) (at 120.3452 77.47 0)
       (effects (font (size 1.27 1.27)) hide)
     )
@@
       (effects (font (size 1.27 1.27)) (justify left))
     )
-    (property "Value" "" (id 1) (at 130.81 82.5499 0)
+    (property "Value" "8-40p" (id 1) (at 130.81 82.5499 0)
       (effects (font (size 1.27 1.27)) (justify left))
     )
-    (property "Footprint" "" (id 2) (at 127.9652 85.09 0)
+    (property "Footprint" "Capacitor_SMD:C_0603_1608Metric" (id 2) (at 127.9652 85.09 0)
       (effects (font (size 1.27 1.27)) hide)
     )
@@
       (effects (font (size 1.27 1.27)) (justify left))
     )
-    (property "Value" "" (id 1) (at 130.81 95.2499 0)
+    (property "Value" "8-40p" (id 1) (at 130.81 95.2499 0)
       (effects (font (size 1.27 1.27)) (justify left))
     )
-    (property "Footprint" "" (id 2) (at 127.9652 97.79 0)
+    (property "Footprint" "Capacitor_SMD:C_0603_1608Metric" (id 2) (at 127.9652 97.79 0)
       (effects (font (size 1.27 1.27)) hide)
     )
@@
     (in_bom yes) (on_board yes) (fields_autoplaced)
     (property "Reference" "R2" (id 0) (at 143.51 91.44 90))
-    (property "Value" "" (id 1) (at 143.51 93.98 90))
-    (property "Footprint" "" (id 2) (at 143.764 96.774 90)
+    (property "Value" "R_US" (id 1) (at 143.51 93.98 90))
+    (property "Footprint" "Resistor_SMD:R_0603_1608Metric" (id 2) (at 143.764 96.774 90)
       (effects (font (size 1.27 1.27)) hide)
     )
@@
     (in_bom yes) (on_board yes)
     (property "Reference" "C4" (id 0) (at 105.41 107.95 90))
-    (property "Value" "" (id 1) (at 105.41 110.49 90))
-    (property "Footprint" "" (id 2) (at 109.22 101.9048 0)
+    (property "Value" "8-40p" (id 1) (at 105.41 110.49 90))
+    (property "Footprint" "Capacitor_SMD:C_0603_1608Metric" (id 2) (at 109.22 101.9048 0)
       (effects (font (size 1.27 1.27)) hide)
     )
@@
       (effects (font (size 1.27 1.27)) (justify right))
     )
-    (property "Value" "" (id 1) (at 115.57 95.2499 0)
+    (property "Value" "30p" (id 1) (at 115.57 95.2499 0)
       (effects (font (size 1.27 1.27)) (justify right))
     )
-    (property "Footprint" "" (id 2) (at 120.3452 90.17 0)
+    (property "Footprint" "Capacitor_SMD:C_0603_1608Metric" (id 2) (at 120.3452 90.17 0)
       (effects (font (size 1.27 1.27)) hide)
     )
@@
     (in_bom yes) (on_board yes) (fields_autoplaced)
     (property "Reference" "R1" (id 0) (at 143.51 71.12 90))
-    (property "Value" "" (id 1) (at 143.51 73.66 90))
-    (property "Footprint" "" (id 2) (at 143.764 76.454 90)
+    (property "Value" "R_US" (id 1) (at 143.51 73.66 90))
+    (property "Footprint" "Resistor_SMD:R_0603_1608Metric" (id 2) (at 143.764 76.454 90)
       (effects (font (size 1.27 1.27)) hide)
     )
@@
     (in_bom yes) (on_board yes) (fields_autoplaced)
     (property "Reference" "C3" (id 0) (at 105.41 90.17 90))
-    (property "Value" "" (id 1) (at 105.41 92.71 90))
-    (property "Footprint" "" (id 2) (at 109.22 96.8248 0)
+    (property "Value" "NC" (id 1) (at 105.41 92.71 90))
+    (property "Footprint" "Capacitor_SMD:C_0603_1608Metric" (id 2) (at 109.22 96.8248 0)
       (effects (font (size 1.27 1.27)) hide)
     )
@@
     (in_bom yes) (on_board yes)
     (property "Reference" "C2" (id 0) (at 105.41 82.55 90))
-    (property "Value" "" (id 1) (at 105.41 85.09 90))
-    (property "Footprint" "" (id 2) (at 109.22 76.5048 0)
-      (effects (font (size 1.27 1.27)) hide)
-    )
+    (property "Value" "NC" (id 1) (at 105.41 85.09 90))
+    (property "Footprint" "Capacitor_SMD:C_0603_1608Metric" (id 2) (at 109.22 76.5048 0)
+      (effects (font (size 1.27 1.27)) hide)
+    )

Commit message: Final rev 1.0.0
Parts:
- C1: value 8-40p -> (none); footprint Resistor_SMD:R_0603_1608Metric -> (none)
- C4, C7, C8: value 8-40p -> (none); footprint Capacitor_SMD:C_0603_1608Metric -> (none)
Changed lines of the file:
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@@
     (in_bom yes) (on_board yes) (fields_autoplaced)
     (property "Reference" "C1" (id 0) (at 105.41 64.77 90))
-    (property "Value" "8-40p" (id 1) (at 105.41 67.31 90))
-    (property "Footprint" "Resistor_SMD:R_0603_1608Metric" (id 2) (at 109.22 71.4248 0)
+    (property "Value" "" (id 1) (at 105.41 67.31 90))
+    (property "Footprint" "" (id 2) (at 109.22 71.4248 0)
       (effects (font (size 1.27 1.27)) hide)
     )
@@
       (effects (font (size 1.27 1.27)) (justify left))
     )
-    (property "Value" "8-40p" (id 1) (at 130.81 82.5499 0)
+    (property "Value" "" (id 1) (at 130.81 82.5499 0)
       (effects (font (size 1.27 1.27)) (justify left))
     )
-    (property "Footprint" "Capacitor_SMD:C_0603_1608Metric" (id 2) (at 127.9652 85.09 0)
+    (property "Footprint" "" (id 2) (at 127.9652 85.09 0)
       (effects (font (size 1.27 1.27)) hide)
     )
@@
       (effects (font (size 1.27 1.27)) (justify left))
     )
-    (property "Value" "8-40p" (id 1) (at 130.81 95.2499 0)
+    (property "Value" "" (id 1) (at 130.81 95.2499 0)
       (effects (font (size 1.27 1.27)) (justify left))
     )
-    (property "Footprint" "Capacitor_SMD:C_0603_1608Metric" (id 2) (at 127.9652 97.79 0)
+    (property "Footprint" "" (id 2) (at 127.9652 97.79 0)
       (effects (font (size 1.27 1.27)) hide)
     )
@@
     (in_bom yes) (on_board yes)
     (property "Reference" "C4" (id 0) (at 105.41 107.95 90))
-    (property "Value" "8-40p" (id 1) (at 105.41 110.49 90))
-    (property "Footprint" "Capacitor_SMD:C_0603_1608Metric" (id 2) (at 109.22 101.9048 0)
+    (property "Value" "" (id 1) (at 105.41 110.49 90))
+    (property "Footprint" "" (id 2) (at 109.22 101.9048 0)
       (effects (font (size 1.27 1.27)) hide)
     )
@@
   (symbol_instances
     (path "/02ab15cc-d4b2-48c5-a9cd-646284b23111"
-      (reference "C1") (unit 1) (value "8-40p") (footprint "Resistor_SMD:R_0603_1608Metric")
+      (reference "C1") (unit 1) (value "11p") (footprint "Resistor_SMD:R_0603_1608Metric")
     )
     (path "/e2e20a04-e569-4b7b-a4f2-db2a07b068bb"
@@
     )
     (path "/a97f35f9-349f-4c3a-b8b8-43d6d23efb6c"
-      (reference "C4") (unit 1) (value "8-40p") (footprint "Capacitor_SMD:C_0603_1608Metric")
+      (reference "C4") (unit 1) (value "11p") (footprint "Capacitor_SMD:C_0603_1608Metric")
     )
     (path "/30827bd8-2c45-4b23-a780-e074789ebb44"
@@
     )
     (path "/57084d4e-a4ea-4ca2-940d-82b7c846897f"
-      (reference "C7") (unit 1) (value "8-40p") (footprint "Capacitor_SMD:C_0603_1608Metric")
+      (reference "C7") (unit 1) (value "32p") (footprint "Capacitor_SMD:C_0603_1608Metric")
     )
     (path "/8adc823a-7fcc-4921-9aae-eafe09355df0"
-      (reference "C8") (unit 1) (value "8-40p") (footprint "Capacitor_SMD:C_0603_1608Metric")
+      (reference "C8") (unit 1) (value "32p") (footprint "Capacitor_SMD:C_0603_1608Metric")
     )
     (path "/2eda4bfe-b50d-4efe-b93a-e95f3e8ce559"
